File: HAND_Project_ADS1220_Amplifier/HAND_Project_ADS1220_Amplifier.kicad_pcb (KiCad board)
At the start: 2 copper layers, 10 parts, among them J1 Screw_Terminal_01x04, J2 Conn_01x03_Pin, J3 Conn_01x03_Pin, U1 ADS1220IPWR

Commit message: After meeting
Parts:
- moved D2 5.68 mm to (119.4, 115.0)
Other:
- board outline added: 30.5 x 38.1 mm
Changed lines of the file:
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@@
 	(footprint "Diode_SMD:D_SMA"
 		(layer "F.Cu")
-		(at 124.46 112.49 90)
+		(at 119.38 115.03 90)
 		(descr "Diode SMA (DO-214AC)")
 		(tags "Diode SMA (DO-214AC)")
@@
 		)
 	)
+	(gr_circle
+		(center 110.49 148.59)
+		(end 110.49 149.86)
+		(stroke
+			(width 0.2)
+			(type default)
+		)
+		(fill no)
+		(layer "F.Cu")
+	)
+	(gr_rect
+		(start 107.95 97.79)
+		(end 138.43 135.89)
+		(stroke
+			(width 0.2)
+			(type solid)
+		)
+		(fill no)
+		(layer "Edge.Cuts")
+	)
 	(embedded_fonts no)
